Commit message: + modified friction coeff.

File: allegro_hand_description/urdf/allegro_hand.gazebo.xacro (robot description, xacro)
@@ -33,4 +33,7 @@
             <provideFeedback>true</provideFeedback>
             <implicitSpringDamper>true</implicitSpringDamper>
+            <stopKd value="1.0" />
+            <stopKp value="1e7" />
+            <fudgeFactor value="1.0" />
         </gazebo>
         <transmission name="${reference}_tran">
@@ -50,8 +53,9 @@
         <gazebo reference="${reference}">
             <!-- <turnGravityOff>true</turnGravityOff> -->
-            <mu1>0.05</mu1>
-            <mu2>0.05</mu2>
+            <mu1>500</mu1>
+            <mu2>500</mu2>
             <!-- This defines the springiness of the contacts: 400000 -->
-            <kp>1000</kp>
+            <kp>1e8</kp>
+            <kd>1.0</kd>
             <selfCollide>false</selfCollide>
             <material>Gazebo/Grey</material>

File: allegro_hand_description/urdf/allegro_hand_description_right.xacro (robot description, xacro)
@@ -74,4 +74,6 @@
     <xacro:property name="joint_damping" value="0.05"/>
     <xacro:property name="joint_friction" value="0.00"/>
+    <xacro:property name="joint_effort" value="100"/> <!-- 15 -->
+    <xacro:property name="joint_velocity" value="100"/> <!-- 7 -->
     <!-- ============================================================================= -->
     <!-- THUMB MACRO -->
@@ -128,5 +130,5 @@
         <joint name="finger_${finger_num}/joint_0" type="revolute">
             <axis xyz="-1 0 0"/>
-            <limit effort="15" velocity="7"
+            <limit effort="${joint_effort}" velocity="${joint_velocity}"
                    lower="${limit_0_t_low + joint_safety_margin}"
                    upper="${limit_0_t_up  - joint_safety_margin}"/>
@@ -180,5 +182,5 @@
         <joint name="finger_${finger_num}/joint_1" type="revolute">
             <axis xyz="0 0 1"/>
-            <limit effort="15" velocity="7"
+            <limit effort="${joint_effort}" velocity="${joint_velocity}"
                    lower="${limit_1_t_low + joint_safety_margin}"
                    upper="${limit_1_t_up  - joint_safety_margin}"/>
@@ -229,5 +231,5 @@
         <joint name="finger_${finger_num}/joint_2" type="revolute">
             <axis xyz="0 1 0"/>
-            <limit effort="15" velocity="7"
+            <limit effort="${joint_effort}" velocity="${joint_velocity}"
                    lower="${limit_2_t_low + joint_safety_margin}"
                    upper="${limit_2_t_up  - joint_safety_margin}"/>
@@ -279,5 +281,5 @@
         <joint name="finger_${finger_num}/joint_3" type="revolute">
             <axis xyz="0 1 0"/>
-            <limit effort="15" velocity="7"
+            <limit effort="${joint_effort}" velocity="${joint_velocity}"
                    lower="${limit_3_t_low + joint_safety_margin}"
                    upper="${limit_3_t_up  - joint_safety_margin}"/>
@@ -390,5 +392,5 @@
         <joint name="finger_${finger_num}/joint_0" type="revolute">
             <axis xyz="0 0 1"/>
-            <limit effort="15" velocity="7"
+            <limit effort="${joint_effort}" velocity="${joint_velocity}"
                    lower="${limit_0_low + joint_safety_margin}"
                    upper="${limit_0_up  - joint_safety_margin}"/>
@@ -439,5 +441,5 @@
         />
         <joint name="finger_${finger_num}/joint_1" type="revolute">
-            <limit effort="15" velocity="7"
+            <limit effort="${joint_effort}" velocity="${joint_velocity}"
                    lower="${limit_1_low + joint_safety_margin}"
                    upper="${limit_1_up  - joint_safety_margin}"/>
@@ -489,5 +491,5 @@
         <joint name="finger_${finger_num}/joint_2" type="revolute">
             <axis xyz="0 1 0"/>
-            <limit effort="15" velocity="7"
+            <limit effort="${joint_effort}" velocity="${joint_velocity}"
                    lower="${limit_2_low + joint_safety_margin}"
                    upper="${limit_2_up  - joint_safety_margin}"/>
@@ -538,5 +540,5 @@
         <joint name="finger_${finger_num}/joint_3" type="revolute">
             <axis xyz="0 1 0"/>
-            <limit effort="15" velocity="7"
+            <limit effort="${joint_effort}" velocity="${joint_velocity}"
                    lower="${limit_3_low + joint_safety_margin}"
                    upper="${limit_3_up  - joint_safety_margin}"/>
